File: Arduino_shield.brd (EAGLE design)
At the start: 240 x 880 mm, 21 parts

Commit message: Initial_handmade_routing
Parts:
- moved DEV8 751.6 mm to (99.7, -25.1)
- moved DEV6 722.5 mm to (76.7, -5.36)
- moved DEV7 722.4 mm to (49.7, -25.2)
- moved DEV4 700.4 mm to (99.7, 14.4)
- moved DEV5 694.5 mm to (25.7, -5.50)
- moved DEV2 671.0 mm to (76.7, 34.1)
- moved DEV3 670.7 mm to (49.7, 14.2)
- moved DEV1 642.6 mm to (25.7, 33.9)
- moved EXTRADIG 612.5 mm to (-70.1, 40.0)
- moved EXTRAANALOGUE 587.9 mm to (-23.3, 0.92), turned to 90 degrees
- moved BUZZER 503.2 mm to (-6.32, -45.6)
- moved REL3 259.7 mm to (-7.68, -6.43)
- moved REL4 253.7 mm to (-7.54, -25.1)
- moved REL1 217.1 mm to (-7.67, 34.1)
- moved TEMP2 201.6 mm to (22.6, 72.7)
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Connections:
- removed net SS5: BONUS.2, U$1.6
- net D1A: now also DEV1.P$2, REL1.6; no longer DEV1.P$3, REL2.6
- net D1B: now also DEV1.P$3, REL1.7; no longer DEV1.P$2, REL2.7
- net D22: now also EXTRADIG.2; no longer EXTRADIG.1
- net D23: now also EXTRADIG.1; no longer EXTRADIG.2
- net D24: now also EXTRADIG.4; no longer EXTRADIG.3
- net D25: now also EXTRADIG.3; no longer EXTRADIG.4
- net D26: now also EXTRADIG.6; no longer EXTRADIG.5
- net D27: now also EXTRADIG.5; no longer EXTRADIG.6
- net D28: now also EXTRADIG.8; no longer EXTRADIG.7
- net D29: now also EXTRADIG.7; no longer EXTRADIG.8
- net D2A: now also DEV2.P$2, REL1.3; no longer DEV2.P$3, REL2.3
- net D2B: now also DEV2.P$3, REL1.2; no longer DEV2.P$2, REL2.2
- net D30: now also EXTRADIG.10; no longer EXTRADIG.9
- net D31: now also EXTRADIG.9; no longer EXTRADIG.10
- net D32: now also EXTRADIG.12; no longer EXTRADIG.11
- net D33: now also EXTRADIG.11; no longer EXTRADIG.12
- net D34: now also EXTRADIG.14; no longer EXTRADIG.13
- net D35: now also EXTRADIG.13; no longer EXTRADIG.14
- net D36: now also EXTRADIG.16; no longer EXTRADIG.15
- net D37: now also EXTRADIG.15; no longer EXTRADIG.16
- net D38: now also EXTRADIG.18; no longer EXTRADIG.17
- net D39: now also EXTRADIG.17; no longer EXTRADIG.18
- net D3A: now also DEV3.P$2, REL2.6; no longer DEV3.P$3, REL1.6
- net D3B: now also DEV3.P$3, REL2.7; no longer DEV3.P$2, REL1.7
- net D40: now also EXTRADIG.20; no longer EXTRADIG.19
- net D41: now also EXTRADIG.19; no longer EXTRADIG.20
- net D42: now also EXTRADIG.22; no longer EXTRADIG.21
- net D43: now also EXTRADIG.21; no longer EXTRADIG.22
- net D44: now also EXTRADIG.24; no longer EXTRADIG.23
- net D45: now also EXTRADIG.23; no longer EXTRADIG.24
- net D46: now also EXTRADIG.26; no longer EXTRADIG.25
- net D47: now also EXTRADIG.25; no longer EXTRADIG.26
- net D48: now also EXTRADIG.28; no longer EXTRADIG.27
- net D49: now also EXTRADIG.27; no longer EXTRADIG.28
- net D4A: now also DEV4.P$2, REL2.3; no longer DEV4.P$3, REL1.3
- net D4B: now also DEV4.P$3, REL2.2; no longer DEV4.P$2, REL1.2
- net D50: now also EXTRADIG.30; no longer EXTRADIG.29
- net D51: now also EXTRADIG.29; no longer EXTRADIG.30
- net D52: now also EXTRADIG.32; no longer EXTRADIG.31
- net D53: now also EXTRADIG.31; no longer EXTRADIG.32
- net D5A: now also DEV5.P$2, REL3.6; no longer DEV5.P$3, REL4.6
- net D5B: now also DEV5.P$3, REL3.7; no longer DEV5.P$2, REL4.7
- net D6A: now also DEV6.P$2, REL3.3; no longer DEV6.P$3, REL4.3
- net D6B: now also DEV6.P$3, REL3.2; no longer DEV6.P$2, REL4.2
- net D7A: now also DEV7.P$2, REL4.6; no longer DEV7.P$3, REL3.6
- net D7B: now also DEV7.P$3, REL4.7; no longer DEV7.P$2, REL3.7
- net D8A: now also DEV8.P$2, REL4.3; no longer DEV8.P$3, REL3.3
- net D8B: now also DEV8.P$3, REL4.2; no longer DEV8.P$2, REL3.2
- net GND: now also U$1.5V_ICSP, U$1.GND1, U$1.GND_2, U$1.GND_A, U$1.GND_B
- net RR1: now also REL2.1; no longer REL1.1
- net RR2: now also REL1.1; no longer REL2.1
- net RR3: now also REL4.1; no longer REL3.1
- net RR4: now also REL3.1; no longer REL4.1
- net SS4: now also BONUS.2
Routing:
- net DOUT: track 0.00 -> 235.3 mm, vias 0 -> 2
- net MISO: track 0.00 -> 199.7 mm
- net SCK: track 0.00 -> 197.1 mm, vias 0 -> 4
- net MOSI: track 0.00 -> 186.4 mm, vias 0 -> 2
- net BDOUT: track 0.00 -> 186.2 mm
- net T1OUT: track 0.00 -> 142.7 mm, vias 0 -> 2
- net D8B: track 0.00 -> 123.1 mm
- net D4B: track 0.00 -> 122.7 mm
- net D8A: track 0.00 -> 115.0 mm
- net D4A: track 0.00 -> 114.6 mm
- net D6B: track 0.00 -> 100.8 mm
- net D2B: track 0.00 -> 100.5 mm
- net D6A: track 0.00 -> 92.8 mm
- net D2A: track 0.00 -> 91.7 mm
- net D3B: track 0.00 -> 72.8 mm
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- added copper zone on layer 1, net GND
- added copper zone on layer 16, net GND
Other:
- board size 240 x 880 mm -> 240 x 160 mm

Commit message: finished_autorouting_no_rules
Routing:
- net SDA: track 38.7 -> 439.6 mm, vias 0 -> 1
- net -15V: track 38.7 -> 432.3 mm, vias 0 -> 1
- net +5V: track 38.7 -> 430.4 mm, vias 0 -> 2
- net +15V: track 38.7 -> 414.1 mm, vias 0 -> 3
- net SCL: track 38.7 -> 380.5 mm, vias 0 -> 2
- net +3V3: track 38.7 -> 369.3 mm, vias 0 -> 2
- net MOSI: track 186.4 -> 462.5 mm
- net SCK: track 197.1 -> 469.1 mm
- net MISO: track 199.7 -> 437.6 mm, vias 0 -> 2
- net SS3: track 0.00 -> 188.2 mm
- net SS2: track 0.00 -> 163.1 mm
- net SS4: track 0.00 -> 147.2 mm
- net AOUT: track 0.00 -> 144.3 mm, vias 0 -> 1
- net T2OUT: track 0.00 -> 143.3 mm
- net RR2: track 0.00 -> 129.2 mm, vias 0 -> 2
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