File: Arduino_shield.brd (EAGLE design)
At the start: 240 x 160 mm, 21 parts

Commit message: finished_ruled_autorouting
Routing:
- net BAOUT: track 128.5 -> 129.7 mm
- net -15V: track 514.4 -> 513.7 mm
Changed lines of the file:
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@@
 <attribute name="OC_NEWARK" value="unknown" x="-77.38" y="73.252" size="1.778" layer="27" display="off"/>
 <attribute name="MF" value="" x="-77.38" y="73.252" size="1.778" layer="27" display="off"/>
-<attribute name="NAME" x="-86.905" y="79.1702" size="0.889" layer="25" ratio="24"/>
+<attribute name="NAME" x="-94.525" y="71.8042" size="0.889" layer="25" ratio="24"/>
 <attribute name="VALUE" x="-87.54" y="66.902" size="1.27" layer="27"/>
 </element>
 <element name="PWR" library="CoilCircuitLibrary_E7" package="6PIN_CON" value="6PIN_CON" x="106.46" y="65.68" smashed="yes" rot="R180">
-<attribute name="NAME" x="109" y="73.3" size="0.889" layer="25" font="vector" ratio="24" rot="R180"/>
+<attribute name="NAME" x="95.284" y="71.014" size="0.889" layer="25" font="vector" ratio="24" rot="R180"/>
 </element>
 <element name="TEMP2" library="con-harting" package="CON16L" value="" x="22.62" y="72.73" smashed="yes">
@@
 <attribute name="OC_NEWARK" value="unknown" x="22.62" y="72.73" size="1.778" layer="27" display="off"/>
 <attribute name="MF" value="" x="22.62" y="72.73" size="1.778" layer="27" display="off"/>
-<attribute name="NAME" x="13.095" y="78.6482" size="0.889" layer="25" ratio="24"/>
+<attribute name="NAME" x="5.475" y="71.7902" size="0.889" layer="25" ratio="24"/>
 <attribute name="VALUE" x="12.46" y="66.38" size="1.27" layer="27"/>
 </element>
@@
 <attribute name="OC_NEWARK" value="unknown" x="78.95" y="-58.62" size="1.778" layer="27" rot="R270" display="off"/>
 <attribute name="MF" value="" x="78.95" y="-58.62" size="1.778" layer="27" rot="R270" display="off"/>
-<attribute name="NAME" x="84.8682" y="-49.095" size="0.889" layer="25" ratio="24" rot="R270"/>
+<attribute name="NAME" x="72.9302" y="-57.477" size="0.889" layer="25" ratio="24" rot="R270"/>
 <attribute name="VALUE" x="72.6" y="-48.46" size="1.27" layer="27" rot="R270"/>
 </element>
@@
 <attribute name="OC_NEWARK" value="unknown" x="41.39" y="-58.62" size="1.778" layer="27" rot="R270" display="off"/>
 <attribute name="MF" value="" x="41.39" y="-58.62" size="1.778" layer="27" rot="R270" display="off"/>
-<attribute name="NAME" x="47.3082" y="-49.095" size="0.889" layer="25" ratio="24" rot="R270"/>
+<attribute name="NAME" x="34.6082" y="-57.477" size="0.889" layer="25" ratio="24" rot="R270"/>
 <attribute name="VALUE" x="35.04" y="-48.46" size="1.27" layer="27" rot="R270"/>
 </element>
@@
 <wire x1="-86.36" y1="72.39" x2="-86.27" y2="71.982" width="0.254" layer="16"/>
 <wire x1="13.97" y1="71.12" x2="13.73" y2="71.46" width="0.254" layer="16"/>
-<wire x1="-21.59" y1="-16.51" x2="-21.59" y2="-15.24" width="0.254" layer="1"/>
 <wire x1="-20.32" y1="-17.78" x2="-21.59" y2="-16.51" width="0.254" layer="1"/>
 <wire x1="-16.51" y1="-13.97" x2="-20.32" y2="-17.78" width="0.254" layer="16"/>
@@
 <wire x1="12.7" y1="55.88" x2="-8.89" y2="34.29" width="0.254" layer="16"/>
 <wire x1="-8.89" y1="34.29" x2="-16.51" y2="26.67" width="0.254" layer="16"/>
-<wire x1="-21.59" y1="-15.24" x2="-21.99" y2="-15.59" width="0.254" layer="1"/>
 <wire x1="24.13" y1="-33.02" x2="40.64" y2="-49.53" width="0.254" layer="1"/>
 <wire x1="-8.89" y1="0" x2="24.13" y2="-33.02" width="0.254" layer="16"/>
@@
 <via x="-20.32" y="-17.78" extent="1-16" drill="0.6096"/>
 <via x="24.13" y="-33.02" extent="1-16" drill="0.6096"/>
+<wire x1="-21.59" y1="-16.51" x2="-21.59" y2="-15.99" width="0.254" layer="1"/>
+<wire x1="-21.59" y1="-15.99" x2="-21.99" y2="-15.59" width="0.254" layer="1"/>
 </signal>
 <signal name="+5V">
@@
 <contactref element="BONUS" pad="8"/>
 <contactref element="U$1" pad="A0"/>
-<wire x1="34.29" y1="-59.69" x2="40.64" y2="-59.69" width="0.254" layer="1"/>
-<wire x1="2.54" y1="-27.94" x2="34.29" y2="-59.69" width="0.254" layer="16"/>
+<wire x1="32.258" y1="-59.69" x2="40.64" y2="-59.69" width="0.254" layer="1"/>
 <wire x1="2.54" y1="-20.32" x2="2.54" y2="-27.94" width="0.254" layer="16"/>
 <wire x1="-10.16" y1="-7.62" x2="2.54" y2="-20.32" width="0.254" layer="16"/>
@@
 <wire x1="40.64" y1="-59.69" x2="40.12" y2="-59.89" width="0.254" layer="1"/>
 <wire x1="-43.18" y1="-30.48" x2="-43.35" y2="-30.25" width="0.254" layer="16"/>
-<via x="34.29" y="-59.69" extent="1-16" drill="0.6096"/>
+<via x="32.258" y="-59.69" extent="1-16" drill="0.6096"/>
+<wire x1="32.258" y1="-59.69" x2="32.258" y2="-57.658" width="0.254" layer="16"/>
+<wire x1="32.258" y1="-57.658" x2="2.54" y2="-27.94" width="0.254" layer="16"/>
 </signal>
 <signal name="BDOUT">
