File: Arduino_shield.brd (EAGLE design)
At the start: 240 x 160 mm, 21 parts

Commit message: ready_to_print
Parts:
- moved DEV1 10.0 mm to (15.7, 33.9)
- moved DEV2 10.0 mm to (66.7, 34.1)
- moved DEV3 10.0 mm to (39.7, 14.2)
- moved DEV4 10.0 mm to (89.7, 14.4)
- moved DEV5 10.0 mm to (15.7, -5.50)
- moved DEV6 10.0 mm to (66.7, -5.36)
- moved DEV7 10.0 mm to (39.7, -25.2)
- moved DEV8 10.0 mm to (89.7, -25.1)
- moved PWR 10.0 mm to (96.5, 65.7)
Routing:
- net +15V: track 499.3 -> 453.1 mm, vias 4 -> 5
- net D3A: track 64.7 -> 54.7 mm
- net D5A: track 40.2 -> 30.2 mm
- net D8B: track 123.1 -> 113.1 mm
- net D8A: track 115.0 -> 105.0 mm
- net D7B: track 72.6 -> 62.6 mm
- net D6B: track 100.8 -> 90.8 mm
- net D6A: track 92.8 -> 82.8 mm
- net D4B: track 122.7 -> 112.7 mm
- net D4A: track 114.6 -> 104.6 mm
- net D2B: track 100.5 -> 90.5 mm
- net D2A: track 91.7 -> 81.7 mm
- net D1B: track 48.0 -> 38.0 mm
- net D1A: track 40.3 -> 30.3 mm
- net D7A: track 64.2 -> 54.2 mm
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Other:
- board size 240 x 160 mm -> 230 x 160 mm

Commit message: production
Routing:
- net SDA: track 398.5 -> 404.5 mm
- net GND: track 6.87 -> 11.5 mm, vias 21 -> 22
- net MISO: track 541.1 -> 544.9 mm
- net +15V: track 453.1 -> 456.9 mm
- net T1OUT: track 142.7 -> 140.6 mm
- net SS3: track 230.7 -> 229.7 mm
- net SCL: track 434.0 -> 433.2 mm
- net BAOUT: track 129.7 -> 130.5 mm
- net SCK: track 443.7 -> 443.0 mm
- net RR1: track 116.8 -> 117.5 mm
- net +3V3: track 348.7 -> 349.2 mm
- net -15V: track 504.7 -> 505.2 mm
Other:
- board text added: "Srylab 05/2022 Arduino Shield Jacopo De Santis v1.0"
- board text removed: "Srylab 03/2022 Arduino_shield Jacopo De Santis v1.0"
